File: KiCad/HKB44.kicad_pcb (KiCad board)
At the start: 2 copper layers, 275.6 x 79.9 mm, 102 parts, among them J1 Conn_01x04_Female, J2 Arduino_pro_micro_conn, SW0 SW_Push, SW1 SW_Push, SW10 SW_Push, SW100 SW_Push, SW11 SW_Push, SW12 SW_Push, SW13 SW_Push, SW14 SW_Push, SW15 SW_Push, SW16 SW_Push, SW2 SW_Push, SW20 SW_Push, SW22 SW_Push, SW23 SW_Push, SW24 SW_Push, SW25 SW_Push, SW26 SW_Push, SW3 SW_Push, SW30 SW_Push, SW31 SW_Push, SW32 SW_Push, SW33 SW_Push, SW34 SW_Push, SW36 SW_Push, SW4 SW_Push, SW40 SW_Push, SW42 SW_Push, SW43 SW_Push, SW44 SW_Push, SW45 SW_Push, SW46 SW_Push, SW5 SW_Push, SW50 SW_Push, SW51 SW_Push, SW52 SW_Push, SW53 SW_Push, SW55 SW_Push, SW6 SW_Push, SW60 SW_Push, SW61 SW_Push, SW62 SW_Push, SW66 SW_Push, SW73 SW_Push, SW74 SW_Push, SW75 SW_Push, SW76 SW_Push

Commit message: HKB43 version 0.9
Parts:
- removed D13, D54: 1N4148, Diode_SMD:D_SOD-323_HandSoldering
- removed the J2 at (69.7, 88.7)
- removed the J2 at (68.4, 86.2)
- removed SW15, SW74: SW_Push, HKB44:MX_PCB_100H
- added J2: Arduino_pro_micro_conn, library:Arduino_pro_micro_conn, B.Cu at (68.4, 85.0)
- added J3: Conn_01x04_Male, Connector_JST:JST_SH_BM04B-SRSS-TB_1x04-1MP_P1.00mm_Vertical, F.Cu at (66.4, 51.1)
- added J4: USB_B_Micro, library:USB_Micro-B_Molex_47346-0001, F.Cu at (53.5, 43.7)
- added REF**: SolderJumper-2_P1.3mm_Open_TrianglePad1.0x1.5mm, Jumper:SolderJumper-2_P1.3mm_Open_TrianglePad1.0x1.5mm, F.Cu at (45.9, 49.3)
- added REF**: MountingHole_3mm_Pad_Via, MountingHole:MountingHole_3mm_Pad_Via, F.Cu at (186.4, 74.2)
- added REF**: MountingHole_3mm_Pad_Via, MountingHole:MountingHole_3mm_Pad_Via, F.Cu at (110.2, 74.2)
- added REF**: MountingHole_3mm_Pad_Via, MountingHole:MountingHole_3mm_Pad_Via, F.Cu at (34.0, 66.5)
- added REF**: USB_Micoro-B-Pad, library:USB_Micoro-B-Pad, B.Cu at (56.1, 46.9)
- added REF**: OSHW-Logo2_9.8x8mm_Copper, Symbol:OSHW-Logo2_9.8x8mm_Copper, B.Cu at (136.8, 129.5)
- added REF**: MountingHole_3mm_Pad_Via, MountingHole:MountingHole_3mm_Pad_Via, F.Cu at (186.4, 53.6)
- added REF**: MountingHole_3mm_Pad_Via, MountingHole:MountingHole_3mm_Pad_Via, F.Cu at (34.0, 46.0)
- added REF**: MountingHole_3mm_Pad_Via, MountingHole:MountingHole_3mm_Pad_Via, F.Cu at (110.2, 53.6)
- added REF**: MountingHole_3mm_Pad_Via, MountingHole:MountingHole_3mm_Pad_Via, F.Cu at (245.9, 46.0)
- added REF**: MountingHole_3mm_Pad_Via, MountingHole:MountingHole_3mm_Pad_Via, F.Cu at (245.9, 66.5)
- SW100: footprint library:B3U-1000P(OMRON Ultra-small Tactile Switch) -> library:push switch; moved to F.Cu
- SW16: footprint HKB44:MX_PCB_100H -> HKB44:MX_PCB_200H
- SW73: footprint HKB44:MX_PCB_100H -> HKB44:MX_PCB_150H
- moved REF** 86.6 mm to (69.3, 54.0)
- moved D14 18.9 mm to (251.7, 73.3), turned to 0 degrees
- moved D11 14.9 mm to (218.8, 77.0), turned to 90 degrees
- moved D12 14.9 mm to (237.9, 77.0), turned to 90 degrees
- moved D8 14.9 mm to (161.7, 77.0), turned to 90 degrees
- moved D9 14.9 mm to (180.7, 77.0), turned to 90 degrees
- moved D10 14.9 mm to (199.8, 77.0), turned to 90 degrees
- moved D6 14.7 mm to (123.5, 76.8), turned to 90 degrees
- moved D1 14.6 mm to (28.3, 76.7), turned to 90 degrees
- moved D4 14.6 mm to (85.4, 76.7), turned to 90 degrees
- moved D5 14.6 mm to (104.5, 76.7), turned to 90 degrees
- moved D7 14.6 mm to (142.6, 76.7), turned to 90 degrees
- moved D3 14.1 mm to (66.5, 76.0), turned to 180 degrees
- moved D2 13.8 mm to (47.0, 75.9), turned to 180 degrees
- moved D55 10.0 mm to (237.0, 121.3)
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Routing:
- net COL6: track 422.3 -> 340.1 mm, vias 5 -> 3
- net COL0: track 278.0 -> 225.7 mm, vias 6 -> 3
- net ROW1: track 262.8 -> 217.0 mm
- net COL4: track 291.9 -> 248.9 mm
- net COL5: track 309.6 -> 272.7 mm
- net COL3: track 280.6 -> 247.4 mm
- net ROW7: track 239.4 -> 206.3 mm
- net ROW0: track 170.9 -> 140.4 mm
- net RST: track 67.1 -> 37.1 mm, vias 2 -> 1
- net VCC: track 321.3 -> 349.9 mm, vias 8 -> 7
- net GND: track 262.6 -> 234.9 mm, vias 14 -> 311
- net USB_VBUS: track 0.00 -> 23.2 mm, vias 0 -> 4
- net ROW6: track 169.1 -> 147.5 mm
- net Net-(J2-Pad3): track 20.2 -> 0.00 mm, vias 1 -> 0
- net LED: track 88.5 -> 68.7 mm
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Other:
- board size 275.6 x 79.9 mm -> 266.4 x 96.7 mm
- board text added: "43"
- board text added: "April 26, 2020 revision 0.9 @hanyazou"
- board text added: "DM"
- board text added: "DP"
- board text added: "HKB43 April 26, 2020 revision 0.9 @hanyazou"
- board text added: "USB"
- board text added: "VBUS"
- board text removed: "45"
- board text removed: "April 19, 2020 revision 0.5 @hanyazou"

Commit message: keyunit x4 key board for POC
Parts:
- removed D10, D11, D12, D14, D15, D17, D18, D19, D20, D21, D22, D23, D24, D25, D26, D28, D29, D3, D31, D32, D33, D34, D35, D36, D37, D38, D39, D4, D41, D43, D44, D45, D49, D5, D53, D55, D56, D6, D7, D8, D9: 1N4148, Diode_SMD:D_SOD-323_HandSoldering
- removed LED3, LED4, LED5, LED6, LED7: WS2812B, library:LED_WS2812B-PLCC4
- removed the REF** at (45.9, 49.3)
- removed the REF** at (186.4, 74.2)
- removed the REF** at (110.2, 74.2)
- removed the REF** at (34.0, 66.5)
- removed the REF** at (56.1, 46.9)
- removed the REF** at (136.8, 129.5)
- removed the REF** at (69.3, 54.0)
- removed the REF** at (186.4, 53.6)
- removed the REF** at (34.0, 46.0)
- removed the REF** at (110.2, 53.6)
- removed the REF** at (245.9, 46.0)
- removed the REF** at (245.9, 66.5)
- removed SW10, SW11, SW12, SW13, SW14, SW2, SW22, SW23, SW24, SW25, SW26, SW3, SW30, SW31, SW32, SW33, SW34, SW4, SW42, SW43, SW44, SW45, SW46, SW5, SW50, SW51, SW52, SW53, SW6, SW75: SW_Push, HKB44:MX_PCB_100H
- removed SW100: SW_Push, library:push switch
- removed SW16: SW_Push, HKB44:MX_PCB_200H
- removed SW20: SW_Push, HKB44:MX_PCB_175H
- removed SW36, SW40: SW_Push, HKB44:MX_PCB_225H
- removed SW55: SW_Push, HKB44:MX_PCB_275H
- removed SW60, SW61, SW62, SW76: SW_Push, HKB44:MX_PCB_125H
- removed SW66: SW_Push, HKB44:MX_PCB_625H
- removed SW73: SW_Push, HKB44:MX_PCB_150H
- added J5: Conn_01x04_Male, Connector_PinHeader_2.54mm:PinHeader_1x04_P2.54mm_Vertical, F.Cu at (40.5, 12.0)
- added J6: Conn_01x04_Male, Connector_PinHeader_2.54mm:PinHeader_1x04_P2.54mm_Vertical, F.Cu at (45.1, 12.0)
- added J7: Conn_01x02_Male, Connector_PinHeader_2.54mm:PinHeader_1x02_P2.54mm_Vertical, F.Cu at (40.5, 24.2)
- added J8: Conn_01x02_Male, Connector_PinHeader_2.54mm:PinHeader_1x02_P2.54mm_Vertical, F.Cu at (49.8, 12.0)
- added JP1: Jumper_NO_Small, Jumper:SolderJumper-2_P1.3mm_Open_TrianglePad1.0x1.5mm, F.Cu at (16.2, 31.4)
- added REF**: MountingHole_3.2mm_M3_Pad_Via, MountingHole:MountingHole_3.2mm_M3_Pad_Via, F.Cu at (15.0, 65.7)
- added REF**: MountingHole_3.2mm_M3_Pad_Via, MountingHole:MountingHole_3.2mm_M3_Pad_Via, F.Cu at (34.0, 65.7)
- added U1: test, library:test, F.Cu at (42.8, 66.5)
- added U2: test, library:test, F.Cu at (49.9, 66.5)
- added U3: test, library:test, F.Cu at (57.1, 66.5)
- added U4: test, library:test, F.Cu at (64.2, 66.5)
- added U5: test, library:test, F.Cu at (42.8, 73.7)
- added U6: test, library:test, F.Cu at (49.9, 73.7)
- added U7: test, library:test, F.Cu at (57.1, 73.7)
- added U8: test, library:test, F.Cu at (64.2, 73.7)
- D2: moved to F.Cu
- J1: value Conn_01x04_Female -> Conn_01x02_Male; footprint Connector_PinHeader_2.54mm:PinHeader_1x04_P2.54mm_Vertical -> Connector_PinHeader_2.54mm:PinHeader_1x02_P2.54mm_Vertical
- J2: value Arduino_pro_micro_conn -> Conn_01x02_Male; footprint library:Arduino_pro_micro_conn -> Connector_PinHeader_2.54mm:PinHeader_1x02_P2.54mm_Vertical; moved to F.Cu
- J3: footprint Connector_JST:JST_SH_BM04B-SRSS-TB_1x04-1MP_P1.00mm_Vertical -> Connector_PinHeader_2.54mm:PinHeader_1x04_P2.54mm_Vertical
- J4: value USB_B_Micro -> Conn_01x04_Male; footprint library:USB_Micro-B_Molex_47346-0001 -> Connector_PinHeader_2.54mm:PinHeader_1x04_P2.54mm_Vertical
- LED1: value WS2812B -> WS2812C-2020; footprint library:LED_WS2812B-PLCC4 -> HKB44:WS2812C2020
- LED2: footprint library:LED_WS2812B-PLCC4 -> LED_SMD:LED_SK6812MINI_PLCC4_3.5x3.5mm_P1.75mm
- SW0, SW1: footprint HKB44:MX_PCB_100H -> HKB44:MX_PCB_100H_socket
- moved LED2 89.6 mm to (46.3, 24.4), turned to 0 degrees
- moved J2 68.9 mm to (35.8, 24.2), turned to 0 degrees
- moved D2 57.3 mm to (11.5, 31.1), turned to 0 degrees
- moved J1 57.1 mm to (31.2, 24.2), turned to 0 degrees
- moved LED1 57.0 mm to (24.5, 62.4), turned to 0 degrees
- moved SW1 56.5 mm to (18.9, 19.6), turned to 0 degrees
- moved J3 52.6 mm to (31.2, 12.0), turned to 0 degrees
- moved J4 36.3 mm to (35.8, 12.0), turned to 0 degrees
- moved D1 10.2 mm to (29.5, 66.5), turned to 270 degrees
- turned SW0 to 0 degrees
Connections:
- J1 pad 1: SDA -> COL0
- J1 pad 2: SCL -> VCC
- J2 pad 1: COL0 -> COL1
- J2 pad 2: LED -> VCC
- J3 pad 1: USB_GND -> ROW0
- J3 pad 2: USB_VBUS -> ROW1
- J3 pad 3: UBS_DP -> LEDIN
- J3 pad 4: USB_DM -> VCC
- J4 pad 1: USB_VBUS -> ROW0
- J4 pad 2: USB_DM -> ROW1
- J4 pad 3: UBS_DP -> LED
- J4 pad 4: Net-(J4-Pad4) -> VCC
- LED1 pad 1: VCC -> LEDOUT
- LED1 pad 2: Net-(LED1-Pad2) -> GND
- LED1 pad 3: GND -> LEDIN
- LED1 pad 4: LED -> VCC
- LED2 pad 4: Net-(LED1-Pad2) -> LED
Routing:
- net COL6: track 340.1 -> 0.00 mm, vias 3 -> 0
- net VCC: track 349.9 -> 48.0 mm
- net COL5: track 272.7 -> 0.00 mm, vias 4 -> 0
- net COL1: track 250.0 -> 0.00 mm, vias 2 -> 0
- net COL4: track 248.9 -> 0.00 mm, vias 3 -> 0
- net COL3: track 247.4 -> 0.00 mm, vias 2 -> 0
- net COL2: track 240.2 -> 0.00 mm, vias 3 -> 0
- net GND: track 234.9 -> 21.6 mm, vias 311 -> 3
- net ROW5: track 212.5 -> 0.00 mm, vias 3 -> 0
- net ROW7: track 206.3 -> 0.00 mm, vias 1 -> 0
- net ROW3: track 205.5 -> 0.00 mm, vias 1 -> 0
- net COL0: track 225.7 -> 26.2 mm, vias 3 -> 2
- net ROW1: track 217.0 -> 18.9 mm, vias 1 -> 3
- net ROW6: track 147.5 -> 0.00 mm, vias 1 -> 0
- net ROW2: track 124.4 -> 0.00 mm, vias 1 -> 0
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- removed copper zone on B.Cu, net GND
- removed copper zone on F.Cu, net GND
Other:
- board size 266.4 x 96.7 mm -> 54.8 x 19.1 mm
- board text removed: "43"
- board text removed: "April 26, 2020 revision 0.9 @hanyazou"
- board text removed: "COL0"
- board text removed: "COL1"
- board text removed: "COL2"
- board text removed: "COL3"
- board text removed: "COL4"
- board text removed: "COL5"
- board text removed: "COL6"
- board text removed: "DM"
- board text removed: "DP"
- board text removed: "GND"
- board text removed: "HKB"
- board text removed: "HKB43 April 26, 2020 revision 0.9 @hanyazou"
- board text removed: "ROW0"
- board text removed: "ROW1"
- board text removed: "ROW2"
- board text removed: "ROW3"
- board text removed: "ROW4"
- board text removed: "ROW5"
- board text removed: "ROW6"
- board text removed: "ROW7"
- board text removed: "SCL"
- board text removed: "SDA"
- board text removed: "USB"
- board text removed: "VBUS"
- board text removed: "VCC"

Commit message: Revert HKB44 board changes
Parts:
- removed J5, J6: Conn_01x04_Male, Connector_PinHeader_2.54mm:PinHeader_1x04_P2.54mm_Vertical
- removed J7, J8: Conn_01x02_Male, Connector_PinHeader_2.54mm:PinHeader_1x02_P2.54mm_Vertical
- removed JP1: Jumper_NO_Small, Jumper:SolderJumper-2_P1.3mm_Open_TrianglePad1.0x1.5mm
- removed the REF** at (15.0, 65.7)
- removed the REF** at (34.0, 65.7)
- removed U1, U2, U3, U4, U5, U6, U7, U8: test, library:test
- added D10: 1N4148, Diode_SMD:D_SOD-323_HandSoldering, B.Cu at (199.8, 77.0)
- added D11: 1N4148, Diode_SMD:D_SOD-323_HandSoldering, B.Cu at (218.8, 77.0)
- added D12: 1N4148, Diode_SMD:D_SOD-323_HandSoldering, B.Cu at (237.9, 77.0)
- added D14: 1N4148, Diode_SMD:D_SOD-323_HandSoldering, B.Cu at (251.7, 73.3)
- added D15: 1N4148, Diode_SMD:D_SOD-323_HandSoldering, B.Cu at (27.9, 83.2)
- added D17: 1N4148, Diode_SMD:D_SOD-323_HandSoldering, B.Cu at (49.8, 87.0)
- added D18: 1N4148, Diode_SMD:D_SOD-323_HandSoldering, B.Cu at (68.8, 87.0)
- added D19: 1N4148, Diode_SMD:D_SOD-323_HandSoldering, B.Cu at (92.1, 83.2)
- added D20: 1N4148, Diode_SMD:D_SOD-323_HandSoldering, B.Cu at (111.2, 83.2)
- added D21: 1N4148, Diode_SMD:D_SOD-323_HandSoldering, B.Cu at (130.2, 83.2)
- added D22: 1N4148, Diode_SMD:D_SOD-323_HandSoldering, B.Cu at (149.3, 83.2)
- added D23: 1N4148, Diode_SMD:D_SOD-323_HandSoldering, B.Cu at (168.3, 83.3)
- added D24: 1N4148, Diode_SMD:D_SOD-323_HandSoldering, B.Cu at (187.4, 83.2)
- added D25: 1N4148, Diode_SMD:D_SOD-323_HandSoldering, B.Cu at (206.4, 83.2)
- added D26: 1N4148, Diode_SMD:D_SOD-323_HandSoldering, B.Cu at (225.5, 83.2)
- added D28: 1N4148, Diode_SMD:D_SOD-323_HandSoldering, B.Cu at (252.0, 87.0)
- added D29: 1N4148, Diode_SMD:D_SOD-323_HandSoldering, B.Cu at (32.6, 102.3)
- added D3: 1N4148, Diode_SMD:D_SOD-323_HandSoldering, B.Cu at (66.5, 76.0)
- added D31: 1N4148, Diode_SMD:D_SOD-323_HandSoldering, B.Cu at (63.6, 102.3)
- added D32: 1N4148, Diode_SMD:D_SOD-323_HandSoldering, B.Cu at (82.6, 102.2)
- added D33: 1N4148, Diode_SMD:D_SOD-323_HandSoldering, B.Cu at (101.7, 102.2)
- added D34: 1N4148, Diode_SMD:D_SOD-323_HandSoldering, B.Cu at (120.7, 102.2)
- added D35: 1N4148, Diode_SMD:D_SOD-323_HandSoldering, B.Cu at (139.8, 102.2)
- added D36: 1N4148, Diode_SMD:D_SOD-323_HandSoldering, B.Cu at (158.8, 102.2)
- added D37: 1N4148, Diode_SMD:D_SOD-323_HandSoldering, B.Cu at (177.9, 102.2)
- added D38: 1N4148, Diode_SMD:D_SOD-323_HandSoldering, B.Cu at (196.9, 102.2)
- added D39: 1N4148, Diode_SMD:D_SOD-323_HandSoldering, B.Cu at (216.0, 102.2)
- added D4: 1N4148, Diode_SMD:D_SOD-323_HandSoldering, B.Cu at (85.4, 76.7)
- added D41: 1N4148, Diode_SMD:D_SOD-323_HandSoldering, B.Cu at (251.6, 102.2)
- added D43: 1N4148, Diode_SMD:D_SOD-323_HandSoldering, B.Cu at (28.5, 121.3)
- added D44: 1N4148, Diode_SMD:D_SOD-323_HandSoldering, B.Cu at (52.4, 121.3)
- added D45: 1N4148, Diode_SMD:D_SOD-323_HandSoldering, B.Cu at (73.1, 121.3)
- added D49: 1N4148, Diode_SMD:D_SOD-323_HandSoldering, B.Cu at (144.5, 121.3)
- added D5: 1N4148, Diode_SMD:D_SOD-323_HandSoldering, B.Cu at (104.5, 76.7)
- added D53: 1N4148, Diode_SMD:D_SOD-323_HandSoldering, B.Cu at (218.4, 121.2)
- added D55: 1N4148, Diode_SMD:D_SOD-323_HandSoldering, B.Cu at (237.0, 121.3)
- added D56: 1N4148, Diode_SMD:D_SOD-323_HandSoldering, B.Cu at (258.5, 121.3)
- added D6: 1N4148, Diode_SMD:D_SOD-323_HandSoldering, B.Cu at (123.5, 76.8)
- added D7: 1N4148, Diode_SMD:D_SOD-323_HandSoldering, B.Cu at (142.6, 76.7)
- added D8: 1N4148, Diode_SMD:D_SOD-323_HandSoldering, B.Cu at (161.7, 77.0)
- added D9: 1N4148, Diode_SMD:D_SOD-323_HandSoldering, B.Cu at (180.7, 77.0)
- added LED3: WS2812B, library:LED_WS2812B-PLCC4, F.Cu at (115.0, 99.1)
- added LED4: WS2812B, library:LED_WS2812B-PLCC4, F.Cu at (134.0, 99.1)
- added LED5: WS2812B, library:LED_WS2812B-PLCC4, F.Cu at (153.1, 99.1)
- added LED6: WS2812B, library:LED_WS2812B-PLCC4, F.Cu at (172.1, 99.1)
- added LED7: WS2812B, library:LED_WS2812B-PLCC4, F.Cu at (191.2, 99.1)
- added REF**: SolderJumper-2_P1.3mm_Open_TrianglePad1.0x1.5mm, Jumper:SolderJumper-2_P1.3mm_Open_TrianglePad1.0x1.5mm, F.Cu at (45.9, 49.3)
- added REF**: MountingHole_3mm_Pad_Via, MountingHole:MountingHole_3mm_Pad_Via, F.Cu at (186.4, 74.2)
- added REF**: MountingHole_3mm_Pad_Via, MountingHole:MountingHole_3mm_Pad_Via, F.Cu at (110.2, 74.2)
- added REF**: MountingHole_3mm_Pad_Via, MountingHole:MountingHole_3mm_Pad_Via, F.Cu at (34.0, 66.5)
- added REF**: USB_Micoro-B-Pad, library:USB_Micoro-B-Pad, B.Cu at (56.1, 46.9)
- added REF**: OSHW-Logo2_9.8x8mm_Copper, Symbol:OSHW-Logo2_9.8x8mm_Copper, B.Cu at (136.8, 129.5)
- added REF**: OSHW-Logo2_9.8x8mm_SilkScreen, Symbol:OSHW-Logo2_9.8x8mm_SilkScreen, B.Cu at (69.3, 54.0)
- added REF**: MountingHole_3mm_Pad_Via, MountingHole:MountingHole_3mm_Pad_Via, F.Cu at (186.4, 53.6)
- added REF**: MountingHole_3mm_Pad_Via, MountingHole:MountingHole_3mm_Pad_Via, F.Cu at (34.0, 46.0)
- added REF**: MountingHole_3mm_Pad_Via, MountingHole:MountingHole_3mm_Pad_Via, F.Cu at (110.2, 53.6)
- added REF**: MountingHole_3mm_Pad_Via, MountingHole:MountingHole_3mm_Pad_Via, F.Cu at (245.9, 46.0)
- added REF**: MountingHole_3mm_Pad_Via, MountingHole:MountingHole_3mm_Pad_Via, F.Cu at (245.9, 66.5)
- added SW10: SW_Push, HKB44:MX_PCB_100H, F.Cu at (157.9, 70.5)
- added SW100: SW_Push, library:push switch, F.Cu at (41.8, 90.2)
- added SW11: SW_Push, HKB44:MX_PCB_100H, F.Cu at (176.9, 70.5)
- added SW12: SW_Push, HKB44:MX_PCB_100H, F.Cu at (196.0, 70.5)
- added SW13: SW_Push, HKB44:MX_PCB_100H, F.Cu at (215.0, 70.5)
- added SW14: SW_Push, HKB44:MX_PCB_100H, F.Cu at (234.1, 70.5)
- added SW16: SW_Push, HKB44:MX_PCB_200H, F.Cu at (262.6, 70.5)
- added SW2: SW_Push, HKB44:MX_PCB_100H, F.Cu at (62.6, 70.5)
- added SW20: SW_Push, HKB44:MX_PCB_175H, F.Cu at (31.6, 89.5)
- added SW22: SW_Push, HKB44:MX_PCB_100H, F.Cu at (57.8, 89.5)
- added SW23: SW_Push, HKB44:MX_PCB_100H, F.Cu at (76.9, 89.5)
- added SW24: SW_Push, HKB44:MX_PCB_100H, F.Cu at (95.9, 89.5)
- added SW25: SW_Push, HKB44:MX_PCB_100H, F.Cu at (115.0, 89.5)
- added SW26: SW_Push, HKB44:MX_PCB_100H, F.Cu at (134.0, 89.5)
- added SW3: SW_Push, HKB44:MX_PCB_100H, F.Cu at (81.7, 70.5)
- added SW30: SW_Push, HKB44:MX_PCB_100H, F.Cu at (153.1, 89.5)
- added SW31: SW_Push, HKB44:MX_PCB_100H, F.Cu at (172.1, 89.5)
- added SW32: SW_Push, HKB44:MX_PCB_100H, F.Cu at (191.2, 89.5)
- added SW33: SW_Push, HKB44:MX_PCB_100H, F.Cu at (210.2, 89.5)
- added SW34: SW_Push, HKB44:MX_PCB_100H, F.Cu at (229.3, 89.5)
- added SW36: SW_Push, HKB44:MX_PCB_225H, F.Cu at (260.3, 89.5)
- added SW4: SW_Push, HKB44:MX_PCB_100H, F.Cu at (100.7, 70.5)
- added SW40: SW_Push, HKB44:MX_PCB_225H, F.Cu at (36.4, 108.6)
- added SW42: SW_Push, HKB44:MX_PCB_100H, F.Cu at (67.4, 108.6)
- added SW43: SW_Push, HKB44:MX_PCB_100H, F.Cu at (86.4, 108.6)
- added SW44: SW_Push, HKB44:MX_PCB_100H, F.Cu at (105.5, 108.6)
- added SW45: SW_Push, HKB44:MX_PCB_100H, F.Cu at (124.5, 108.6)
- added SW46: SW_Push, HKB44:MX_PCB_100H, F.Cu at (143.6, 108.6)
- added SW5: SW_Push, HKB44:MX_PCB_100H, F.Cu at (119.8, 70.5)
- added SW50: SW_Push, HKB44:MX_PCB_100H, F.Cu at (162.6, 108.6)
- added SW51: SW_Push, HKB44:MX_PCB_100H, F.Cu at (181.7, 108.6)
- added SW52: SW_Push, HKB44:MX_PCB_100H, F.Cu at (200.7, 108.6)
- added SW53: SW_Push, HKB44:MX_PCB_100H, F.Cu at (219.8, 108.6)
- added SW55: SW_Push, HKB44:MX_PCB_275H, F.Cu at (255.5, 108.6)
- added SW6: SW_Push, HKB44:MX_PCB_100H, F.Cu at (138.8, 70.5)
- added SW60: SW_Push, HKB44:MX_PCB_125H, F.Cu at (29.3, 127.6)
- added SW61: SW_Push, HKB44:MX_PCB_125H, F.Cu at (53.1, 127.6)
- added SW62: SW_Push, HKB44:MX_PCB_125H, F.Cu at (76.9, 127.6)
- added SW66: SW_Push, HKB44:MX_PCB_625H, F.Cu at (148.3, 127.6)
- added SW73: SW_Push, HKB44:MX_PCB_150H, F.Cu at (222.2, 127.6)
- added SW75: SW_Push, HKB44:MX_PCB_100H, F.Cu at (246.0, 127.6)
- added SW76: SW_Push, HKB44:MX_PCB_125H, F.Cu at (267.4, 127.6)
- D2: moved to B.Cu
- J1: value Conn_01x02_Male -> Conn_01x04_Female; footprint Connector_PinHeader_2.54mm:PinHeader_1x02_P2.54mm_Vertical -> Connector_PinHeader_2.54mm:PinHeader_1x04_P2.54mm_Vertical
- J2: value Conn_01x02_Male -> Arduino_pro_micro_conn; footprint Connector_PinHeader_2.54mm:PinHeader_1x02_P2.54mm_Vertical -> library:Arduino_pro_micro_conn; moved to B.Cu
- J3: footprint Connector_PinHeader_2.54mm:PinHeader_1x04_P2.54mm_Vertical -> Connector_JST:JST_SH_BM04B-SRSS-TB_1x04-1MP_P1.00mm_Vertical
- J4: value Conn_01x04_Male -> USB_B_Micro; footprint Connector_PinHeader_2.54mm:PinHeader_1x04_P2.54mm_Vertical -> library:USB_Micro-B_Molex_47346-0001
- LED1: value WS2812C-2020 -> WS2812B; footprint HKB44:WS2812C2020 -> library:LED_WS2812B-PLCC4
- LED2: footprint LED_SMD:LED_SK6812MINI_PLCC4_3.5x3.5mm_P1.75mm -> library:LED_WS2812B-PLCC4
- SW0, SW1: footprint HKB44:MX_PCB_100H_socket -> HKB44:MX_PCB_100H
- moved LED2 89.6 mm to (95.9, 99.1), turned to 180 degrees
- moved J2 68.9 mm to (68.4, 85.0), turned to 180 degrees
- moved D2 57.3 mm to (47.0, 75.9), turned to 180 degrees
- moved J1 57.1 mm to (37.9, 81.0), turned to 90 degrees
- moved LED1 57.0 mm to (36.5, 118.1), turned to 180 degrees
- moved SW1 56.5 mm to (43.6, 70.5), turned to 180 degrees
- moved J3 52.6 mm to (66.4, 51.1), turned to 270 degrees
- moved J4 36.3 mm to (53.5, 43.7), turned to 270 degrees
- moved D1 10.2 mm to (28.3, 76.7), turned to 90 degrees
- turned SW0 to 180 degrees
Connections:
- J1 pad 1: COL0 -> SDA
- J1 pad 2: VCC -> SCL
- J2 pad 1: COL1 -> COL0
- J2 pad 2: VCC -> LED
- J3 pad 1: ROW0 -> USB_GND
- J3 pad 2: ROW1 -> USB_VBUS
- J3 pad 3: LEDIN -> UBS_DP
- J3 pad 4: VCC -> USB_DM
- J4 pad 1: ROW0 -> USB_VBUS
- J4 pad 2: ROW1 -> USB_DM
- J4 pad 3: LED -> UBS_DP
- J4 pad 4: VCC -> Net-(J4-Pad4)
- LED1 pad 1: LEDOUT -> VCC
- LED1 pad 2: GND -> Net-(LED1-Pad2)
- LED1 pad 3: LEDIN -> GND
- LED1 pad 4: VCC -> LED
- LED2 pad 4: LED -> Net-(LED1-Pad2)
Routing:
- net COL6: track 0.00 -> 340.1 mm, vias 0 -> 3
- net VCC: track 48.0 -> 349.9 mm
- net COL5: track 0.00 -> 272.7 mm, vias 0 -> 4
- net COL1: track 0.00 -> 250.0 mm, vias 0 -> 2
- net COL4: track 0.00 -> 248.9 mm, vias 0 -> 3
- net COL3: track 0.00 -> 247.4 mm, vias 0 -> 2
- net COL2: track 0.00 -> 240.2 mm, vias 0 -> 3
- net GND: track 21.6 -> 234.9 mm, vias 3 -> 311
- net ROW5: track 0.00 -> 212.5 mm, vias 0 -> 3
- net ROW7: track 0.00 -> 206.3 mm, vias 0 -> 1
- net ROW3: track 0.00 -> 205.5 mm, vias 0 -> 1
- net COL0: track 26.2 -> 225.7 mm, vias 2 -> 3
- net ROW1: track 18.9 -> 217.0 mm, vias 3 -> 1
- net ROW6: track 0.00 -> 147.5 mm, vias 0 -> 1
- net ROW2: track 0.00 -> 124.4 mm, vias 0 -> 1
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- added copper zone on B.Cu, net GND
- added copper zone on F.Cu, net GND
Other:
- board size 54.8 x 19.1 mm -> 266.4 x 96.7 mm
- board text added: "43"
- board text added: "April 26, 2020 revision 0.9 @hanyazou"
- board text added: "COL0"
- board text added: "COL1"
- board text added: "COL2"
- board text added: "COL3"
- board text added: "COL4"
- board text added: "COL5"
- board text added: "COL6"
- board text added: "DM"
- board text added: "DP"
- board text added: "GND"
- board text added: "HKB"
- board text added: "HKB43 April 26, 2020 revision 0.9 @hanyazou"
- board text added: "ROW0"
- board text added: "ROW1"
- board text added: "ROW2"
- board text added: "ROW3"
- board text added: "ROW4"
- board text added: "ROW5"
- board text added: "ROW6"
- board text added: "ROW7"
- board text added: "SCL"
- board text added: "SDA"
- board text added: "USB"
- board text added: "VBUS"
- board text added: "VCC"
