File: KiCad/HKB44.sch (KiCad schematic (older format))
At the start: 122 parts, among them J1 Conn_01x04_Female, J2 Arduino_pro_micro_conn, SW0 SW_Push, SW1 SW_Push, SW10 SW_Push, SW100 SW_Push, SW11 SW_Push, SW12 SW_Push, SW13 SW_Push, SW14 SW_Push, SW15 SW_Push, SW16 SW_Push, SW2 SW_Push, SW20 SW_Push, SW21 SW_Push, SW22 SW_Push, SW23 SW_Push, SW24 SW_Push, SW25 SW_Push, SW26 SW_Push, SW3 SW_Push, SW30 SW_Push, SW31 SW_Push, SW32 SW_Push, SW33 SW_Push, SW34 SW_Push, SW35 SW_Push, SW36 SW_Push, SW4 SW_Push, SW40 SW_Push, SW41 SW_Push, SW42 SW_Push, SW43 SW_Push, SW44 SW_Push, SW45 SW_Push, SW46 SW_Push, SW5 SW_Push, SW50 SW_Push, SW51 SW_Push, SW52 SW_Push, SW53 SW_Push, SW54 SW_Push, SW55 SW_Push, SW56 SW_Push, SW6 SW_Push, SW60 SW_Push, SW61 SW_Push, SW62 SW_Push, SW63 SW_Push, SW64 SW_Push, SW65 SW_Push, SW66 SW_Push, SW70 SW_Push, SW71 SW_Push, SW72 SW_Push, SW73 SW_Push, SW74 SW_Push, SW75 SW_Push, SW76 SW_Push

Commit message: HKB43 version 0.9
Parts:
- added J3: Conn_01x04_Male, Connector_JST:JST_SH_BM04B-SRSS-TB_1x04-1MP_P1.00mm_Vertical, symbol Connector:Conn_01x04_Male
- added J4: USB_B_Micro, library:USB_Micro-B_Molex_47346-0001, symbol Connector:USB_B_Micro
- SW100: footprint library:B3U-1000P(OMRON Ultra-small Tactile Switch) -> library:push switch
- SW16: footprint HKB44:MX_PCB_100H -> HKB44:MX_PCB_200H
- SW73: footprint HKB44:MX_PCB_100H -> HKB44:MX_PCB_150H
Connections:
- net labels added: UBS_DP, USB_DM, USB_GND, USB_VBUS
- wire segments 138 -> 140
- no-connect marks 4 -> 6
Other:
- moved on the sheet: J2
Changed lines of the file:
@@
 Text GLabel 1700 5650 0    50   Input ~ 0
 ROW7
-Text GLabel 7900 3900 0    50   Input ~ 0
+Text GLabel 7900 4850 0    50   Input ~ 0
 COL0
-Text GLabel 9300 4800 2    50   Input ~ 0
+Text GLabel 9300 5750 2    50   Input ~ 0
 COL1
-Text GLabel 9300 4700 2    50   Input ~ 0
+Text GLabel 9300 5650 2    50   Input ~ 0
 COL2
-Text GLabel 9300 4600 2    50   Input ~ 0
+Text GLabel 9300 5550 2    50   Input ~ 0
 COL3
-Text GLabel 9300 4500 2    50   Input ~ 0
+Text GLabel 9300 5450 2    50   Input ~ 0
 COL4
-Text GLabel 9300 4400 2    50   Input ~ 0
+Text GLabel 9300 5350 2    50   Input ~ 0
 COL5
-Text GLabel 9300 4300 2    50   Input ~ 0
+Text GLabel 9300 5250 2    50   Input ~ 0
 COL6
-Text GLabel 7900 5000 0    50   Input ~ 0
+Text GLabel 7900 5950 0    50   Input ~ 0
 ROW0
-Text GLabel 7900 4900 0    50   Input ~ 0
+Text GLabel 7900 5850 0    50   Input ~ 0
 ROW1
-Text GLabel 7900 4800 0    50   Input ~ 0
+Text GLabel 7900 5750 0    50   Input ~ 0
 ROW2
-Text GLabel 7900 4700 0    50   Input ~ 0
+Text GLabel 7900 5650 0    50   Input ~ 0
 ROW3
-Text GLabel 7900 4600 0    50   Input ~ 0
+Text GLabel 7900 5550 0    50   Input ~ 0
 ROW4
-Text GLabel 7900 4500 0    50   Input ~ 0
+Text GLabel 7900 5450 0    50   Input ~ 0
 ROW5
-Text GLabel 7900 4400 0    50   Input ~ 0
+Text GLabel 7900 5350 0    50   Input ~ 0
 ROW6
-Text GLabel 7900 4300 0    50   Input ~ 0
+Text GLabel 7900 5250 0    50   Input ~ 0
 ROW7
 $Comp
@@
 	1    0    0    -1
 $EndComp
-Text GLabel 7900 4000 0    50   Input ~ 0
+Text GLabel 7900 4950 0    50   Input ~ 0
 LED
 Text GLabel 1550 6850 0    50   Input ~ 0
@@
 F 0 "SW100" H 8550 2185 50  0000 C CNN
 F 1 "SW_Push" H 8550 2094 50  0000 C CNN
-F 2 "library:B3U-1000P(OMRON Ultra-small Tactile Switch)" H 8550 2100 50  0001 C CNN
+F 2 "library:push switch" H 8550 2100 50  0001 C CNN
 F 3 "" H 8550 2100 50  0001 C CNN
 	1    8550 1900
@@
 Text GLabel 8350 1900 0    50   Input ~ 0
 RST
-Text GLabel 9300 4100 2    50   Input ~ 0
+Text GLabel 9300 5050 2    50   Input ~ 0
 RST
 Wire Wire Line
@@
 	5700 7150 5100 7150
 Connection ~ 5100 7150
-Text GLabel 9300 5000 2    50   Input ~ 0
+Text GLabel 9300 5950 2    50   Input ~ 0
 SDA
-Text GLabel 9300 4900 2    50   Input ~ 0
+Text GLabel 9300 5850 2    50   Input ~ 0
 SCL
 Text GLabel 8450 2500 0    50   Input ~ 0
@@
 F 0 "SW16" H 5700 2050 50  0000 C CNN
 F 1 "SW_Push" H 5700 2044 50  0001 C CNN
-F 2 "HKB44:MX_PCB_100H" H 5700 2050 50  0001 C CNN
+F 2 "HKB44:MX_PCB_200H" H 5700 2050 50  0001 C CNN
 F 3 "" H 5700 2050 50  0001 C CNN
 	1    5700 1850
@@
 F 0 "SW73" H 3900 5650 50  0000 C CNN
 F 1 "SW_Push" H 3900 5644 50  0001 C CNN
-F 2 "HKB44:MX_PCB_100H" H 3900 5650 50  0001 C CNN
+F 2 "HKB44:MX_PCB_150H" H 3900 5650 50  0001 C CNN
 F 3 "" H 3900 5650 50  0001 C CNN
 	1    3900 5450
@@
 	10000 1650 9900 1650
 NoConn ~ 6000 6850
-NoConn ~ 9300 3900
+NoConn ~ 9300 4850
 Text GLabel 1550 6550 0    50   Input ~ 0
 VCC
@@
 Wire Wire Line
 	10600 1650 10600 1500
-Text GLabel 9300 4200 2    50   Input ~ 0
+Text GLabel 9300 5150 2    50   Input ~ 0
 VCC
-Text GLabel 9300 4000 2    50   Input ~ 0
+Text GLabel 9300 4950 2    50   Input ~ 0
 GND
-NoConn ~ 7900 4100
-Text GLabel 7900 4200 0    50   Input ~ 0
+NoConn ~ 7900 5050
+Text GLabel 7900 5150 0    50   Input ~ 0
 GND
 $Comp
 L mylib:Arduino_pro_micro_conn J2
 U 1 1 5EC88007
-P 8600 4250
-F 0 "J2" H 8600 4847 60  0000 C CNN
-F 1 "Arduino_pro_micro_conn" H 8600 4741 60  0000 C CNN
-F 2 "library:Arduino_pro_micro_conn" H 8350 4250 60  0001 C CNN
-F 3 "" H 8350 4250 60  0001 C CNN
-	1    8600 4250
-	1    0    0    -1
-$EndComp
+P 8600 5200
+F 0 "J2" H 8600 5797 60  0000 C CNN
+F 1 "Arduino_pro_micro_conn" H 8600 5691 60  0000 C CNN
+F 2 "library:Arduino_pro_micro_conn" H 8350 5200 60  0001 C CNN
+F 3 "" H 8350 5200 60  0001 C CNN
+	1    8600 5200
+	1    0    0    -1
+$EndComp
+$Comp
+L Connector:Conn_01x04_Male J3
+U 1 1 5EA577FD
+P 9950 2650
+F 0 "J3" H 10058 2931 50  0000 C CNN
+F 1 "Conn_01x04_Male" H 10058 2840 50  0000 C CNN
+F 2 "Connector_JST:JST_SH_BM04B-SRSS-TB_1x04-1MP_P1.00mm_Vertical" H 9950 2650 50  0001 C CNN
+F 3 "~" H 9950 2650 50  0001 C CNN
+	1    9950 2650
+	1    0    0    -1
+$EndComp
+Text GLabel 10150 2650 2    50   Input ~ 0
+USB_VBUS
+Text GLabel 10150 2550 2    50   Input ~ 0
+USB_GND
+Text GLabel 10150 2750 2    50   Input ~ 0
+UBS_DP
+Text GLabel 10150 2850 2    50   Input ~ 0
+USB_DM
+Text GLabel 10150 3800 2    50   Input ~ 0
+USB_DM
+Text GLabel 10150 3700 2    50   Input ~ 0
+UBS_DP
+Text GLabel 10150 3500 2    50   Input ~ 0
+USB_VBUS
+Text GLabel 9900 4200 2    50   Input ~ 0
+USB_GND
+$Comp
+L Connector:USB_B_Micro J4
+U 1 1 5EA7D1A2
+P 9850 3700
+F 0 "J4" H 9907 4167 50  0000 C CNN
+F 1 "USB_B_Micro" H 9907 4076 50  0000 C CNN
+F 2 "library:USB_Micro-B_Molex_47346-0001" H 10000 3650 50  0001 C CNN
+F 3 "~" H 10000 3650 50  0001 C CNN
+	1    9850 3700
+	1    0    0    -1
+$EndComp
+NoConn ~ 9750 4100
+Wire Wire Line
+	9900 4200 9850 4200
+Wire Wire Line
+	9850 4200 9850 4100
+NoConn ~ 10150 3900
 $EndSCHEMATC

Commit message: keyunit x4 key board for POC
Parts:
- SW0, SW1, SW10, SW11, SW12, SW13, SW14, SW15, SW2, SW21, SW22, SW23, SW24, SW25, SW26, SW3, SW30, SW31, SW32, SW33, SW34, SW35, SW4, SW41, SW42, SW43, SW44, SW45, SW46, SW5, SW50, SW51, SW52, SW53, SW54, SW56, SW6, SW63, SW64, SW65, SW70, SW71, SW72, SW74, SW75: footprint HKB44:MX_PCB_100H -> HKB44:MX_PCB_100H_socket
- SW16: footprint HKB44:MX_PCB_200H -> HKB44:MX_PCB_200H_socket
- SW20: footprint HKB44:MX_PCB_175H -> HKB44:MX_PCB_175H_socket
- SW36, SW40: footprint HKB44:MX_PCB_225H -> HKB44:MX_PCB_225H_socket
- SW55: footprint HKB44:MX_PCB_275H -> HKB44:MX_PCB_275H_socket
- SW60, SW61, SW62, SW76: footprint HKB44:MX_PCB_125H -> HKB44:MX_PCB_125H_socket
- SW66: footprint HKB44:MX_PCB_625H -> HKB44:MX_PCB_625H_socket
- SW73: footprint HKB44:MX_PCB_150H -> HKB44:MX_PCB_150H_socket

Commit message: Revert HKB44 board changes
Parts:
- SW0, SW1, SW10, SW11, SW12, SW13, SW14, SW15, SW2, SW21, SW22, SW23, SW24, SW25, SW26, SW3, SW30, SW31, SW32, SW33, SW34, SW35, SW4, SW41, SW42, SW43, SW44, SW45, SW46, SW5, SW50, SW51, SW52, SW53, SW54, SW56, SW6, SW63, SW64, SW65, SW70, SW71, SW72, SW74, SW75: footprint HKB44:MX_PCB_100H_socket -> HKB44:MX_PCB_100H
- SW16: footprint HKB44:MX_PCB_200H_socket -> HKB44:MX_PCB_200H
- SW20: footprint HKB44:MX_PCB_175H_socket -> HKB44:MX_PCB_175H
- SW36, SW40: footprint HKB44:MX_PCB_225H_socket -> HKB44:MX_PCB_225H
- SW55: footprint HKB44:MX_PCB_275H_socket -> HKB44:MX_PCB_275H
- SW60, SW61, SW62, SW76: footprint HKB44:MX_PCB_125H_socket -> HKB44:MX_PCB_125H
- SW66: footprint HKB44:MX_PCB_625H_socket -> HKB44:MX_PCB_625H
- SW73: footprint HKB44:MX_PCB_150H_socket -> HKB44:MX_PCB_150H
