File: KiCad/plate.kicad_pcb (KiCad board)
At the start: 2 copper layers, 266.4 x 76.1 mm, 11 parts

Commit message: Add cherry mx plat footprint and fix HKB44 plate board
Parts:
- removed the REF** at (208.7, 131.1)
- removed the REF** at (105.5, 91.1)
- removed the REF** at (200.7, 91.1)
- added 125u: PLATE, HKB44:MX_PLATE_125H, F.Cu at (267.4, 127.6)
- added 125u: PLATE, HKB44:MX_PLATE_125H, F.Cu at (243.6, 127.6)
- added 125u: PLATE, HKB44:MX_PLATE_125H, F.Cu at (219.8, 127.6)
- added 125u: PLATE, HKB44:MX_PLATE_125H, F.Cu at (76.9, 127.6)
- added 125u: PLATE, HKB44:MX_PLATE_125H, F.Cu at (53.1, 127.6)
- added 125u: PLATE, HKB44:MX_PLATE_125H, F.Cu at (29.3, 127.6)
- added 150u: PLATE, HKB44:MX_PLATE_150H, F.Cu at (267.4, 70.5)
- added 150u: PLATE, HKB44:MX_PLATE_150H, F.Cu at (29.3, 70.5)
- added 175u: PLATE, HKB44:MX_PLATE_175H, F.Cu at (265.0, 108.6)
- added 175u: PLATE, HKB44:MX_PLATE_175H, F.Cu at (31.7, 89.5)
- added 225u: PLATE, HKB44:MX_PLATE_225H, F.Cu at (36.4, 108.6)
- added 225u: PLATE, HKB44:MX_PLATE_225H, F.Cu at (260.3, 89.5)
- added 625u: PLATE, HKB44:MX_PLATE_625H, F.Cu at (148.3, 127.6)
- added REF**: OSHW-Logo2_7.3x6mm_SilkScreen, Symbol:OSHW-Logo2_7.3x6mm_SilkScreen, F.Cu at (164.2, 121.3)
- added REF**: MountingHole_2.2mm_M2_Pad_Via, MountingHole:MountingHole_2.2mm_M2_Pad_Via, F.Cu at (143.6, 99.1)
- added SW1: PLATE, HKB44:MX_PLATE_100H, F.Cu at (67.4, 108.6)
- added SW1: PLATE, HKB44:MX_PLATE_100H, F.Cu at (181.7, 108.6)
- added SW1: PLATE, HKB44:MX_PLATE_100H, F.Cu at (57.8, 89.5)
- added SW1: PLATE, HKB44:MX_PLATE_100H, F.Cu at (115.0, 89.5)
- added SW1: PLATE, HKB44:MX_PLATE_100H, F.Cu at (210.2, 89.5)
- added SW1: PLATE, HKB44:MX_PLATE_100H, F.Cu at (95.9, 89.5)
- added SW1: PLATE, HKB44:MX_PLATE_100H, F.Cu at (229.3, 89.5)
- added SW1: PLATE, HKB44:MX_PLATE_100H, F.Cu at (134.0, 89.5)
- added SW1: PLATE, HKB44:MX_PLATE_100H, F.Cu at (153.1, 89.5)
- added SW1: PLATE, HKB44:MX_PLATE_100H, F.Cu at (191.2, 89.5)
- added SW1: PLATE, HKB44:MX_PLATE_100H, F.Cu at (76.9, 89.5)
- added SW1: PLATE, HKB44:MX_PLATE_100H, F.Cu at (124.5, 108.6)
- added SW1: PLATE, HKB44:MX_PLATE_100H, F.Cu at (172.1, 89.5)
- added SW1: PLATE, HKB44:MX_PLATE_100H, F.Cu at (243.6, 70.5)
- added SW1: PLATE, HKB44:MX_PLATE_100H, F.Cu at (224.5, 70.5)
- added SW1: PLATE, HKB44:MX_PLATE_100H, F.Cu at (205.5, 70.5)
- added SW1: PLATE, HKB44:MX_PLATE_100H, F.Cu at (186.4, 70.5)
- added SW1: PLATE, HKB44:MX_PLATE_100H, F.Cu at (167.4, 70.5)
- added SW1: PLATE, HKB44:MX_PLATE_100H, F.Cu at (148.3, 70.5)
- added SW1: PLATE, HKB44:MX_PLATE_100H, F.Cu at (129.3, 70.5)
- added SW1: PLATE, HKB44:MX_PLATE_100H, F.Cu at (110.2, 70.5)
- added SW1: PLATE, HKB44:MX_PLATE_100H, F.Cu at (91.2, 70.5)
- added SW1: PLATE, HKB44:MX_PLATE_100H, F.Cu at (219.8, 108.6)
- added SW1: PLATE, HKB44:MX_PLATE_100H, F.Cu at (72.1, 70.5)
- added SW1: PLATE, HKB44:MX_PLATE_100H, F.Cu at (53.1, 70.5)
- added SW1: PLATE, HKB44:MX_PLATE_100H, F.Cu at (143.6, 108.6)
- added SW1: PLATE, HKB44:MX_PLATE_100H, F.Cu at (105.5, 108.6)
- added SW1: PLATE, HKB44:MX_PLATE_100H, F.Cu at (162.6, 108.6)
- added SW1: PLATE, HKB44:MX_PLATE_100H, F.Cu at (86.4, 108.6)
- added SW1: PLATE, HKB44:MX_PLATE_100H, F.Cu at (200.7, 108.6)
- added SW1: PLATE, HKB44:MX_PLATE_100H, F.Cu at (238.8, 108.6)
- moved REF** 79.3 mm to (207.9, 118.1)
- moved REF** 59.5 mm to (88.8, 118.1)
- moved REF** 16.7 mm to (277.7, 64.9)
- moved REF** 16.7 mm to (19.0, 64.9)
- moved REF** 9.56 mm to (215.0, 64.9)
- moved REF** 9.56 mm to (81.7, 64.9)
- moved REF** 1.12 mm to (277.7, 133.2)
- moved REF** 1.12 mm to (19.0, 133.2)
Other:
- board size 266.4 x 76.1 mm -> 266.7 x 76.2 mm
- board text added: "HKB44"
- board text removed: "43"
- board text removed: "HKB"
- board text removed: "May 5, 2020 revision 1.00 @hanyazou"
