File: KiCad/keyunit44_plate.kicad_pcb (KiCad board)
At the start: 2 copper layers, 266.7 x 76.2 mm, 54 parts, among them SW1 PLATE

Commit message: Fixed
Parts:
- removed the REF** at (19.0, 64.9)
- removed the REF** at (153.1, 104.1)
- removed the REF** at (215.0, 64.9)
- removed the REF** at (207.9, 118.1)
- removed the REF** at (81.7, 64.9)
- removed the REF** at (88.8, 118.1)
- removed the REF** at (277.7, 133.2)
- removed the REF** at (277.7, 64.9)
- removed the REF** at (19.0, 133.2)
- added REF**: MountingHole_2.2mm_M2, MountingHole:MountingHole_2.2mm_M2, F.Cu at (19.0, 64.9)
- added REF**: MountingHole_2.2mm_M2, MountingHole:MountingHole_2.2mm_M2, F.Cu at (277.7, 133.2)
- added REF**: MountingHole_2.2mm_M2, MountingHole:MountingHole_2.2mm_M2, F.Cu at (207.9, 118.1)
- added REF**: MountingHole_2.2mm_M2, MountingHole:MountingHole_2.2mm_M2, F.Cu at (153.1, 104.1)
- added REF**: MountingHole_2.2mm_M2, MountingHole:MountingHole_2.2mm_M2, F.Cu at (88.8, 118.1)
- added REF**: MountingHole_2.2mm_M2, MountingHole:MountingHole_2.2mm_M2, F.Cu at (19.0, 133.2)
- added REF**: MountingHole_2.2mm_M2, MountingHole:MountingHole_2.2mm_M2, F.Cu at (277.7, 64.9)
- added REF**: MountingHole_2.2mm_M2, MountingHole:MountingHole_2.2mm_M2, F.Cu at (215.0, 64.9)
- added REF**: MountingHole_2.2mm_M2, MountingHole:MountingHole_2.2mm_M2, F.Cu at (81.7, 64.9)
