File: KiCad/keyunit44.kicad_pcb (KiCad board)
At the start: 2 copper layers, 266.7 x 99.2 mm, 70 parts, among them J1 USB_B_Micro, J2 Arduino_pro_micro_conn, J3 Conn_01x04_Female, J4 Conn_01x04_Male, SW1 SW_Push, U11 keyunit, U12 keyunit, U13 keyunit, U14 keyunit, U15 keyunit, U16 keyunit, U17 keyunit, U21 keyunit, U22 keyunit, U23 keyunit, U24 keyunit, U25 keyunit, U26 keyunit, U31 keyunit, U32 keyunit, U33 keyunit, U34 keyunit, U35 keyunit, U36 keyunit, U37 keyunit, U41 keyunit, U42 keyunit, U43 keyunit, U44 keyunit, U46 keyunit, U51 keyunit, U53 keyunit, U54 keyunit, U55 keyunit, U56 keyunit, U57 keyunit, U61 keyunit, U62 keyunit, U63 keyunit, U64 keyunit, U65 keyunit, U66 keyunit, U71 keyunit, U72 keyunit, U73 keyunit, U77 keyunit, U84 keyunit, U85 keyunit, U86 keyunit

Commit message: Output gerber and add .zip files
Routing:
- net Net-(J1-Pad6): vias 16 -> 0
- net GND: vias 175 -> 212
- net (no net): vias 23 -> 2
Other:
- board text added: "HKB44-KU Revision 0.8 November 8, 2020 @hanyazou"
- board text added: "KU Revision 0.8 November 8, 2020 @hanyazou"
- board text removed: "HKB44 Revision 0.9 November 8, 2020 @hanyazou"
- board text removed: "Revision 0.9 November 8, 2020 @hanyazou"

Commit message: Fix keyunit44 version 1.0
Parts:
- removed the REF** at (41.2, 64.9)
- removed the REF** at (255.5, 64.9)
- removed the REF** at (255.5, 41.9)
- removed the REF** at (41.2, 41.9)
- removed the REF** at (119.8, 56.2)
- removed the REF** at (176.9, 56.2)
- removed the REF** at (176.9, 79.2)
- removed the REF** at (119.8, 79.2)
- added REF**: MountingHole_3.2mm_M3, MountingHole:MountingHole_3.2mm_M3, F.Cu at (255.5, 64.9)
- added REF**: MountingHole_3.2mm_M3, MountingHole:MountingHole_3.2mm_M3, F.Cu at (119.8, 56.2)
- added REF**: MountingHole_3.2mm_M3, MountingHole:MountingHole_3.2mm_M3, F.Cu at (176.9, 79.2)
- added REF**: MountingHole_3.2mm_M3, MountingHole:MountingHole_3.2mm_M3, F.Cu at (119.8, 79.2)
- added REF**: MountingHole_3.2mm_M3, MountingHole:MountingHole_3.2mm_M3, F.Cu at (255.5, 41.9)
- added REF**: MountingHole_3.2mm_M3, MountingHole:MountingHole_3.2mm_M3, F.Cu at (176.9, 56.2)
- added REF**: MountingHole_3.2mm_M3, MountingHole:MountingHole_3.2mm_M3, F.Cu at (41.2, 64.9)
- added REF**: MountingHole_3.2mm_M3, MountingHole:MountingHole_3.2mm_M3, F.Cu at (41.2, 41.9)
- J2: footprint library:Arduino_pro_micro_conn -> library:Arduino_pro_micro_0.85mm
Routing:
- net GND: track 718.7 -> 721.9 mm
- net (no net): vias 2 -> 1
Other:
- board text added: "HKB44-KU Revision 1.0 November 28, 2020 @hanyazou"
- board text added: "KU Revision 1.0 November 28, 2020 @hanyazou"
- board text removed: "HKB44-KU Revision 0.8 November 8, 2020 @hanyazou"
- board text removed: "KU Revision 0.8 November 8, 2020 @hanyazou"
