File: KiCad/keyunit44.sch (KiCad schematic (older format))
At the start: 49 parts, among them J1 USB_B_Micro, J2 Arduino_pro_micro_conn, J3 Conn_01x04_Female, J4 Conn_01x04_Male, SW1 SW_Push, U11 keyunit, U12 keyunit, U13 keyunit, U14 keyunit, U15 keyunit, U16 keyunit, U17 keyunit, U21 keyunit, U22 keyunit, U23 keyunit, U24 keyunit, U25 keyunit, U26 keyunit, U31 keyunit, U32 keyunit, U33 keyunit, U34 keyunit, U35 keyunit, U36 keyunit, U37 keyunit, U41 keyunit, U42 keyunit, U43 keyunit, U44 keyunit, U46 keyunit, U51 keyunit, U53 keyunit, U54 keyunit, U55 keyunit, U56 keyunit, U57 keyunit, U61 keyunit, U62 keyunit, U63 keyunit, U64 keyunit, U65 keyunit, U66 keyunit, U71 keyunit, U72 keyunit, U73 keyunit, U77 keyunit, U84 keyunit, U85 keyunit, U86 keyunit

Commit message: Fix keyunit44 version 1.0
Parts:
- J2: footprint library:Arduino_pro_micro_conn -> library:Arduino_pro_micro_0.85mm
Changed lines of the file:
@@
 F 0 "J2" H 8800 5797 60  0000 C CNN
 F 1 "Arduino_pro_micro_conn" H 8800 5691 60  0000 C CNN
-F 2 "library:Arduino_pro_micro_conn" H 8550 5200 60  0001 C CNN
+F 2 "library:Arduino_pro_micro_0.85mm" H 8550 5200 60  0001 C CNN
 F 3 "" H 8550 5200 60  0001 C CNN
 	1    8800 5200
